File: Schematic/V2/overhead/overhead.kicad_pcb (KiCad board)
At the start: 2 copper layers, 50 x 60 mm, 46 parts, among them IC1 74LVC2T45DC,125, J1 PJ-031C, J2 I2C, J3 GPIO, J4 Neopixel 1, J5 Neopixel 2, J6 Micro-USB, J7 Select Jumper, J8 STRAPPING, J9 JTAG, SW1 SW_DIP_x01, SW2 SW_DIP_x01, U1 MIC5528-3.3YMT-TR, U2 ESP32-S2-WROOM, U3 PI3USB221EZWEX, U4 QFN20_SIL, Y1 32.768 kHz

Commit message: uploaded code
Parts:
- removed C8: 2.2 uF, Capacitor_SMD:C_0603_1608Metric_Pad1.08x0.95mm_HandSolder
- removed C9: 100 uF, Capacitor_THT:CP_Radial_D5.0mm_P2.00mm
- removed IC1: 74LVC2T45DC,125, HIVE-Level-Shifter:SOP50P310X100-8N
- removed R5: 10k, Resistor_SMD:R_0805_2012Metric_Pad1.20x1.40mm_HandSolder
- added C13: 100 uF, Capacitor_THT:CP_Radial_D5.0mm_P2.00mm, F.Cu at (67.8, 102.5)
- added REF**: MountingHole_2.2mm_M2, MountingHole:MountingHole_2.2mm_M2, F.Cu at (75.5, 53.2)
- added REF**: MountingHole_2.2mm_M2, MountingHole:MountingHole_2.2mm_M2, F.Cu at (58.0, 87.5)
- added REF**: MountingHole_2.2mm_M2, MountingHole:MountingHole_2.2mm_M2, F.Cu at (101.5, 103.0)
- added U5: NTB0102, Package_SO:TSSOP-8_3x3mm_P0.65mm, F.Cu at (61.8, 102.2)
- C12: footprint Capacitor_SMD:C_0603_1608Metric_Pad1.08x0.95mm_HandSolder -> Capacitor_SMD:C_1206_3216Metric_Pad1.33x1.80mm_HandSolder
- C2, C3: value 12.5 pF -> 7 pF
- C4: footprint Capacitor_SMD:C_1206_3216Metric_Pad1.33x1.80mm_HandSolder -> Capacitor_SMD:C_0805_2012Metric_Pad1.18x1.45mm_HandSolder
- C7: value 2.2 uF -> 10 uF; footprint Capacitor_SMD:C_0603_1608Metric_Pad1.08x0.95mm_HandSolder -> Capacitor_SMD:C_0805_2012Metric_Pad1.18x1.45mm_HandSolder
- D4: footprint HIVE-TVS-Diodes:SOT143 -> Package_TO_SOT_SMD:SOT-553
- J6: value Micro-USB -> 10118193-0001LF; footprint HIVE-micro-usb:10118193-0001LF -> HIVE-finalmicrousb:FCI_10118193-0001LF
- U1: value MIC5528-3.3YMT-TR -> NCP1117ST33T3G; footprint HIVE-linear-regulator:MIC5528-3.3YMT-TR -> HIVE-linreg:SOT230P700X180-4N
- U4: value QFN20_SIL -> CP2102N-A02-GQFN20R; moved to F.Cu
- Y1: value 32.768 kHz -> MS3V-T1R; footprint HIVE-Crystal-Oscillator:ABS25-32.000KHZ-T -> HIVE-finaloscillator:XTAL_MS3V-T1R
- moved R3 56.6 mm to (61.5, 105.5)
- moved C1 55.6 mm to (58.0, 103.8)
- moved C2 4.34 mm to (87.5, 69.1)
- moved C4 3.54 mm to (95.5, 60.5), turned to 0 degrees
- moved U1 3.35 mm to (97.0, 65.5), turned to 180 degrees
- moved U4 2.36 mm to (64.8, 67.5), turned to 90 degrees
- moved C3 2.06 mm to (83.5, 69.0)
- moved Y1 1.53 mm to (85.5, 66.5), turned to 0 degrees
- moved C7 1.50 mm to (99.5, 60.5), turned to 0 degrees
- moved J6 1.12 mm to (62.0, 51.5)
- moved C6 1.00 mm to (93.5, 96.5)
- moved C11 0.50 mm to (60.0, 63.2)
- moved SW1 0.50 mm to (60.0, 94.0)
- turned D4 to 0 degrees
Connections:
- C7 pad 1: +5V -> GND
- C7 pad 2: GND -> +5V
- D4 pad 1: GND -> VBUS
- D4 pad 2: VBUS -> GND
- D4 pad 3: USB)D- -> USB)D+
- D4 pad 4: USB)D+ -> USB)D-
- R3 pad 1: +5V -> Net-(R3-Pad1)
- R3 pad 2: EN -> +3V3
- U1 pad 1: +3V3 -> GND
- U1 pad 3: GND -> +5V
- U1 pad 4: EN -> +3V3
- Y1 pad 1: /XTAL_P -> /XTAL_N
- Y1 pad 2: GND -> /XTAL_P
Routing:
- net +3V3: track 13.6 -> 222.1 mm, vias 6 -> 7
- net ESP32)D-: track 0.00 -> 31.9 mm
- net ESP32)D+: track 0.00 -> 31.9 mm
- net GND: track 24.3 -> 6.12 mm, vias 6 -> 27
- net DIN2: track 38.9 -> 55.6 mm
- net Neopixel1: track 60.9 -> 69.3 mm
- net UART)D+: track 2.43 -> 10.7 mm, vias 1 -> 2
- net UART)D-: track 2.93 -> 10.9 mm, vias 1 -> 2
- net Net-(R3-Pad1): track 0.00 -> 5.16 mm
- net /VSens: track 10.9 -> 8.00 mm, vias 1 -> 0
- net USB)D-: track 13.8 -> 16.4 mm
- net Net-(IC1-Pad5): track 2.49 -> 0.00 mm
- net DIN1: track 13.6 -> 16.0 mm, vias 0 -> 1
- net Neopixel2: track 63.5 -> 61.3 mm
- net EN: track 1.75 -> 0.00 mm
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- removed copper zone on F.Cu, net /XTAL_N
- removed copper zone on F.Cu, net /XTAL_P
Other:
- rule trace_min: 0.2032 -> 0.15
- board text added: "3v3"
- board text added: "5v"
- board text added: "DIN"
- board text added: "GND"
- board text added: "HIVE Lights v1"
- board text added: "MTCK"
- board text added: "MTDI"
- board text added: "MTDO"
- board text added: "SDA SCL"
- board text added: "select"
