File: Schematic/V2/overhead/overhead.sch (KiCad schematic (older format))
At the start: 46 parts, among them IC1 74LVC2T45DC,125, J1 PJ-031C, J2 I2C, J3 GPIO, J4 Neopixel 1, J5 Neopixel 2, J6 Micro-USB, J7 Select Jumper, J8 STRAPPING, J9 JTAG, SW1 SW_DIP_x01, SW2 SW_DIP_x01, U1 MIC5528-3.3YMT-TR, U2 ESP32-S2-WROOM, U3 PI3USB221EZWEX, U4 CP2102N-A02-GQFN20R, Y1 32.768 kHz

Commit message: uploaded code
Parts:
- removed C8: 2.2 uF, Capacitor_SMD:C_0603_1608Metric_Pad1.08x0.95mm_HandSolder, symbol Device:C
- removed C9: 100 uF, Capacitor_THT:CP_Radial_D5.0mm_P2.00mm, symbol Device:C
- removed IC1: 74LVC2T45DC,125, HIVE-Level-Shifter:SOP50P310X100-8N, symbol HIVE-lvl-shifter:74LVC2T45DC,125
- removed J6: Micro-USB, HIVE-micro-usb:10118193-0001LF, symbol HIVE-Micro-USB:10118193-0001LF
- removed R3: 10k, Resistor_SMD:R_0805_2012Metric_Pad1.20x1.40mm_HandSolder, symbol Device:R
- removed R5: 10k, Resistor_SMD:R_0805_2012Metric_Pad1.20x1.40mm_HandSolder, symbol Device:R_US
- removed U1: MIC5528-3.3YMT-TR, HIVE-linear-regulator:MIC5528-3.3YMT-TR, symbol HIVE-Lin-Reg:MIC5528-3.3YMT-TR
- removed Y1: 32.768 kHz, HIVE-Crystal-Oscillator:ABS25-32.000KHZ-T, symbol Device:Crystal_GND23
- added C13: 100 uF, Capacitor_THT:CP_Radial_D5.0mm_P2.00mm, symbol Device:C
- added J6: 10118193-0001LF, HIVE-finalmicrousb:FCI_10118193-0001LF, symbol HIVE-mUSB:10118193-0001LF
- added R3: 10k, Resistor_SMD:R_0805_2012Metric_Pad1.20x1.40mm_HandSolder, symbol Device:R_US
- added U1: NCP1117ST33T3G, HIVE-linreg:SOT230P700X180-4N, symbol HIVE-linreg:NCP1117ST33T3G
- added U5: NTB0102, Package_SO:TSSOP-8_3x3mm_P0.65mm, symbol HIVE-lvl-shifter:NTB0102
- added Y1: MS3V-T1R, HIVE-finaloscillator:XTAL_MS3V-T1R, symbol HIVE-cry-osc:MS3V-T1R
- C12: footprint Capacitor_SMD:C_0603_1608Metric_Pad1.08x0.95mm_HandSolder -> Capacitor_SMD:C_1206_3216Metric_Pad1.33x1.80mm_HandSolder
- C2, C3: value 12.5 pF -> 7 pF
- C4: footprint Capacitor_SMD:C_1206_3216Metric_Pad1.33x1.80mm_HandSolder -> Capacitor_SMD:C_0805_2012Metric_Pad1.18x1.45mm_HandSolder
- C7: value 2.2 uF -> 10 uF; footprint Capacitor_SMD:C_0603_1608Metric_Pad1.08x0.95mm_HandSolder -> Capacitor_SMD:C_0805_2012Metric_Pad1.18x1.45mm_HandSolder
- D4: footprint HIVE-TVS-Diodes:SOT143 -> Package_TO_SOT_SMD:SOT-553
Connections:
- net +3V3: now also R3.2, U1.2 (OUT), U1.4 (OUT), U5.3 (VCCA)
- net +5V: now also C7.2, C13.1, U1.3 (IN), U5.7 (VCCB); no longer C7.1
- net DIN1: now also U5.8 (B1)
- net DIN2: now also U5.1 (B2)
- net GND: now also C7.1, C13.2, J6.5 (GND), J6.S1 (SHIELD), J6.S2 (SHIELD), J6.S3 (SHIELD), J6.S4 (SHIELD), J6.S5 (SHIELD), J6.S6 (SHIELD), U1.1 (GND), U5.2 (GND); no longer C7.2
- net Neopixel1: now also U5.5 (A1)
- net Neopixel2: now also U5.4 (A2)
- net USB)D+: now also J6.3 (D+)
- net USB)D-: now also J6.2 (D-)
- net VBUS: now also J6.1 (VUSB)
- net XTAL_N: now also Y1.1
- net XTAL_P: now also Y1.2
- new net: R3.1, U5.6 (OE)
Other:
- note removed: "*put near lin. reg."
- moved on the sheet: C4, C7, J1
